Commit message: change name from shin to knee

File: opr_description/urdf/version3/legs/left_leg.urdf.xacro (robot description, xacro)
@@ -39,5 +39,5 @@
         <axis xyz="0 0 1" />
     </joint>
-    <joint name="left_knee_pitch_joint" type="revolute" >
+    <joint name="left_knee_pitch_mimic_joint" type="revolute" >
         <parent link="left_waist_pitch_link" />
         <child link="left_knee_pitch_link" />
@@ -47,5 +47,5 @@
         <axis xyz="0 0 1" />
     </joint>
-    <joint name="left_shin_pitch_joint" type="revolute" >
+    <joint name="left_knee_pitch_joint" type="revolute" >
         <parent link="left_knee_pitch_link" />
         <child link="left_shin_pitch_link" />
@@ -58,5 +58,5 @@
         <child link="left_shin_pitch_mimic_link" />
         <origin xyz="0.037 0.032 0" rpy="0 0 0" />
-        <mimic joint="left_shin_pitch_joint" multiplier="1" offset="0" />
+        <mimic joint="left_knee_pitch_joint" multiplier="1" offset="0" />
         <limit effort="1000" lower="${-PI/6}" upper="${PI/2}" velocity="1.0" />
         <axis xyz="0 0 1" />
@@ -66,5 +66,5 @@
         <child link="left_independent_pitch_link" />
         <origin xyz="0.1 0 0" rpy="0 0 0" />
-        <mimic joint="left_shin_pitch_joint" multiplier="-1" offset="0" />
+        <mimic joint="left_knee_pitch_joint" multiplier="-1" offset="0" />
         <limit effort="1000" lower="${-PI/6}" upper="${PI/2}" velocity="1.0" />
         <axis xyz="0 0 1" />

File: opr_description/urdf/version3/legs/right_leg.urdf.xacro (robot description, xacro)
@@ -39,5 +39,5 @@
         <axis xyz="0 0 1" />
     </joint>
-    <joint name="right_knee_pitch_joint" type="revolute" >
+    <joint name="right_knee_pitch_mimic_joint" type="revolute" >
         <parent link="right_waist_pitch_link" />
         <child link="right_knee_pitch_link" />
@@ -47,5 +47,5 @@
         <axis xyz="0 0 1" />
     </joint>
-    <joint name="right_shin_pitch_joint" type="revolute" >
+    <joint name="right_knee_pitch_joint" type="revolute" >
         <parent link="right_knee_pitch_link" />
         <child link="right_shin_pitch_link" />
@@ -58,5 +58,5 @@
         <child link="right_shin_pitch_mimic_link" />
         <origin xyz="0.037 0.032 0" rpy="0 0 0" />
-        <mimic joint="right_shin_pitch_joint" multiplier="1" offset="0" />
+        <mimic joint="right_knee_pitch_joint" multiplier="1" offset="0" />
         <limit effort="1000" lower="${-PI/6}" upper="${PI/2}" velocity="1.0" />
         <axis xyz="0 0 1" />
@@ -66,5 +66,5 @@
         <child link="right_independent_pitch_link" />
         <origin xyz="0.1 0 0" rpy="0 0 0" />
-        <mimic joint="right_shin_pitch_joint" multiplier="-1" offset="0" />
+        <mimic joint="right_knee_pitch_joint" multiplier="-1" offset="0" />
         <limit effort="1000" lower="${-PI/6}" upper="${PI/2}" velocity="1.0" />
         <axis xyz="0 0 1" />
