Commit message: modify files to move on gazebo

File: opr_description/robots/gankenkun_v3.xacro (robot description, xacro)
@@ -7,5 +7,6 @@
     <!-- import empty link -->
     <link name="base_link"/>
-    <!-- uncomment this part to fixed the body in space (ignore gravity)
+    <!-- uncomment this part to fixed the body in space (ignore gravity) -->
+    <!--
     <link name="world"/>
     <joint name="world2base" type="fixed">
@@ -25,4 +26,14 @@
     <xacro:include filename="$(find opr_description)/urdf/version3/sensors/imu/imu.urdf.xacro"/>
     <!-- Import transmission -->
+    <xacro:include filename="$(find opr_description)/urdf/version3/head/head.transmission.xacro"/>
+    <xacro:include filename="$(find opr_description)/urdf/version3/arms/arm.transmission.xacro"/>
+    <xacro:include filename="$(find opr_description)/urdf/version3/legs/leg.transmission.xacro"/>
     <!-- Import gazebo plugin -->
+    <xacro:include filename="$(find opr_description)/urdf/gazebo.xacro"/>
+    <xacro:include filename="$(find opr_description)/urdf/version3/body/body.gazebo.xacro"/>
+    <xacro:include filename="$(find opr_description)/urdf/version3/head/head.gazebo.xacro"/>
+    <xacro:include filename="$(find opr_description)/urdf/version3/arms/arm.gazebo.xacro"/>
+    <xacro:include filename="$(find opr_description)/urdf/version3/legs/leg.gazebo.xacro"/>
+    <xacro:include filename="$(find opr_description)/urdf/version3/sensors/camera/camera.gazebo.xacro"/>
+    <xacro:include filename="$(find opr_description)/urdf/version3/sensors/imu/imu.gazebo.xacro"/>
 </robot>

File: opr_description/urdf/gazebo.xacro (robot description, xacro)
@@ -4,4 +4,5 @@
         <plugin name="gazebo_ros_control" filename="libgazebo_ros_control.so">
             <robotNamespace></robotNamespace>
+            <legacyModeNS>true</legacyModeNS>
         </plugin>
     </gazebo>

File: opr_description/urdf/version3/arms/left_arm.urdf.xacro (robot description, xacro)
@@ -13,5 +13,5 @@
         <child link="left_arm_link" />
         <origin xyz="0 0 0.0315" rpy="0 ${PI/2} 0" />
-        <limit effort="1000" lower="${-PI}" upper="${PI}" velocity="1.0" />
+        <limit effort="1000" lower="0" upper="${PI}" velocity="1.0" />
         <axis xyz="0 0 1" />
     </joint>

File: opr_description/urdf/version3/arms/right_arm.urdf.xacro (robot description, xacro)
@@ -13,5 +13,5 @@
         <child link="right_arm_link" />
         <origin xyz="0 0 -0.0315" rpy="0 ${PI/2} 0" />
-        <limit effort="1000" lower="${-PI}" upper="${PI}" velocity="1.0" />
+        <limit effort="1000" lower="${-PI}" upper="0" velocity="1.0" />
         <axis xyz="0 0 1" />
     </joint>

File: opr_description/urdf/version3/legs/left_leg.urdf.xacro (robot description, xacro)
@@ -21,5 +21,5 @@
         <origin xyz="-0.018 0 -0.091475" rpy="0 0 0" />
         <mimic joint="left_waist_roll_joint" multiplier="-2" offset="0" />
-        <limit effort="1000" lower="${-PI/4}" upper="${PI/4}" velocity="1.0" />
+        <limit effort="1000" lower="${-PI/2}" upper="${PI/2}" velocity="2.0" />
         <axis xyz="0 0 1" />
     </joint>
@@ -67,5 +67,5 @@
         <origin xyz="0.1 0 0" rpy="0 0 0" />
         <mimic joint="left_knee_pitch_joint" multiplier="-1" offset="0" />
-        <limit effort="1000" lower="${-PI/6}" upper="${PI/2}" velocity="1.0" />
+        <limit effort="1000" lower="${-PI/2}" upper="${PI/2}" velocity="1.0" />
         <axis xyz="0 0 1" />
     </joint>

File: opr_description/urdf/version3/legs/right_leg.urdf.xacro (robot description, xacro)
@@ -21,5 +21,5 @@
         <origin xyz="-0.018 0 -0.091475" rpy="0 0 0" />
         <mimic joint="right_waist_roll_joint" multiplier="-2" offset="0" />
-        <limit effort="1000" lower="${-PI/4}" upper="${PI/4}" velocity="1.0" />
+        <limit effort="1000" lower="${-PI/2}" upper="${PI/2}" velocity="2.0" />
         <axis xyz="0 0 1" />
     </joint>
@@ -67,5 +67,5 @@
         <origin xyz="0.1 0 0" rpy="0 0 0" />
         <mimic joint="right_knee_pitch_joint" multiplier="-1" offset="0" />
-        <limit effort="1000" lower="${-PI/6}" upper="${PI/2}" velocity="1.0" />
+        <limit effort="1000" lower="${-PI/2}" upper="${PI/2}" velocity="1.0" />
         <axis xyz="0 0 1" />
     </joint>
