Commit message: change joint name

File: opr_description/urdf/version3/arms/arm.gazebo.xacro (robot description, xacro)
@@ -13,8 +13,8 @@
     </xacro:macro>
     <xacro:arm_reference name="left_shoulder_link"/>
-    <xacro:arm_reference name="left_arm_link"/>
-    <xacro:arm_reference name="left_hand_link"/>
+    <xacro:arm_reference name="left_upper_arm_link"/>
+    <xacro:arm_reference name="left_lower_arm_link"/>
     <xacro:arm_reference name="right_shoulder_link"/>
-    <xacro:arm_reference name="right_arm_link"/>
-    <xacro:arm_reference name="right_hand_link"/>
+    <xacro:arm_reference name="right_upper_arm_link"/>
+    <xacro:arm_reference name="right_lower_arm_link"/>
 </robot>

File: opr_description/urdf/version3/arms/arm.transmission.xacro (robot description, xacro)
@@ -13,9 +13,9 @@
         </transmission>
     </xacro:macro>
-    <xacro:arm_transmission name="left_shoulder"/>
-    <xacro:arm_transmission name="left_arm"/>
-    <xacro:arm_transmission name="left_hand"/>
-    <xacro:arm_transmission name="right_shoulder"/>
-    <xacro:arm_transmission name="right_arm"/>
-    <xacro:arm_transmission name="right_hand"/>
+    <xacro:arm_transmission name="left_shoulder_pitch"/>
+    <xacro:arm_transmission name="left_shoulder_roll"/>
+    <xacro:arm_transmission name="left_elbow_pitch"/>
+    <xacro:arm_transmission name="right_shoulder_pitch"/>
+    <xacro:arm_transmission name="right_shoulder_roll"/>
+    <xacro:arm_transmission name="right_elbow_pitch"/>
 </robot>

File: opr_description/urdf/version3/arms/left_arm.urdf.xacro (robot description, xacro)
@@ -2,5 +2,5 @@
 <robot xmlns:xacro="http://www.ros.org/wiki/xacro">
     <!-- arm joints -->
-    <joint name="left_shoulder_joint" type="revolute" >
+    <joint name="left_shoulder_pitch_joint" type="revolute" >
         <parent link="body_link" />
         <child link="left_shoulder_link" />
@@ -9,14 +9,14 @@
         <axis xyz="0 0 1" />
     </joint>
-    <joint name="left_arm_joint" type="revolute" >
+    <joint name="left_shoulder_roll_joint" type="revolute" >
         <parent link="left_shoulder_link" />
-        <child link="left_arm_link" />
+        <child link="left_upper_arm_link" />
         <origin xyz="0 0 0.0315" rpy="0 ${PI/2} 0" />
         <limit effort="1000" lower="0" upper="${PI}" velocity="1.0" />
         <axis xyz="0 0 1" />
     </joint>
-    <joint name="left_hand_joint" type="revolute" >
-        <parent link="left_arm_link" />
-        <child link="left_hand_link" />
+    <joint name="left_elbow_pitch_joint" type="revolute" >
+        <parent link="left_upper_arm_link" />
+        <child link="left_lower_arm_link" />
         <origin xyz="0 0.109 0" rpy="0 ${-PI/2} 0" />
         <limit effort="1000" lower="${-3*PI/4}" upper="${3*PI/4}" velocity="1.0" />
@@ -44,5 +44,5 @@
         </collision>
     </link>
-    <link name="left_arm_link">
+    <link name="left_upper_arm_link">
         <inertial>
             <mass value="0.185658"/>
@@ -63,5 +63,5 @@
         </collision>
     </link>
-    <link name="left_hand_link">
+    <link name="left_lower_arm_link">
         <inertial>
             <mass value="0.059757"/>

File: opr_description/urdf/version3/arms/right_arm.urdf.xacro (robot description, xacro)
@@ -2,5 +2,5 @@
 <robot xmlns:xacro="http://www.ros.org/wiki/xacro">
     <!-- arm joints -->
-    <joint name="right_shoulder_joint" type="revolute" >
+    <joint name="right_shoulder_pitch_joint" type="revolute" >
         <parent link="body_link" />
         <child link="right_shoulder_link" />
@@ -9,14 +9,14 @@
         <axis xyz="0 0 1" />
     </joint>
-    <joint name="right_arm_joint" type="revolute" >
+    <joint name="right_shoulder_roll_joint" type="revolute" >
         <parent link="right_shoulder_link" />
-        <child link="right_arm_link" />
+        <child link="right_upper_arm_link" />
         <origin xyz="0 0 -0.0315" rpy="0 ${PI/2} 0" />
         <limit effort="1000" lower="${-PI}" upper="0" velocity="1.0" />
         <axis xyz="0 0 1" />
     </joint>
-    <joint name="right_hand_joint" type="revolute" >
-        <parent link="right_arm_link" />
-        <child link="right_hand_link" />
+    <joint name="right_elbow_pitch_joint" type="revolute" >
+        <parent link="right_upper_arm_link" />
+        <child link="right_lower_arm_link" />
         <origin xyz="0 0.109 0" rpy="0 ${-PI/2} 0" />
         <limit effort="1000" lower="${-3*PI/4}" upper="${3*PI/4}" velocity="1.0" />
@@ -44,5 +44,5 @@
         </collision>
     </link>
-    <link name="right_arm_link">
+    <link name="right_upper_arm_link">
         <inertial>
             <mass value="0.185658"/>
@@ -63,5 +63,5 @@
         </collision>
     </link>
-    <link name="right_hand_link">
+    <link name="right_lower_arm_link">
         <inertial>
             <mass value="0.059757"/>
