Commit message: lighter model

File: opr_description/urdf/version3/arms/left_arm.urdf.xacro (robot description, xacro)
@@ -33,5 +33,5 @@
             <origin xyz="0 0 0" rpy="0 0 ${PI/2}"/>
             <geometry>
-                <mesh filename="package://opr_description/meshes/version3/DAE/shoulder.dae" />
+                <mesh filename="package://opr_description/meshes/version3/STL/shoulder.stl" />
             </geometry>
         </visual>
@@ -53,5 +53,5 @@
             <origin xyz="0 0 0" rpy="0 ${PI/2} 0"/>
             <geometry>
-                <mesh filename="package://opr_description/meshes/version3/DAE/arm.dae" />
+                <mesh filename="package://opr_description/meshes/version3/STL/arm.stl" />
             </geometry>
         </visual>
@@ -72,5 +72,5 @@
             <origin xyz="0 0 0" rpy="0 0 ${PI/2}"/>
             <geometry>
-                <mesh filename="package://opr_description/meshes/version3/DAE/hand.dae" />
+                <mesh filename="package://opr_description/meshes/version3/STL/hand.stl" />
             </geometry>
         </visual>

File: opr_description/urdf/version3/arms/right_arm.urdf.xacro (robot description, xacro)
@@ -33,5 +33,5 @@
             <origin xyz="0 0 0" rpy="0 ${PI} ${PI/2}"/>
             <geometry>
-                <mesh filename="package://opr_description/meshes/version3/DAE/shoulder.dae" />
+                <mesh filename="package://opr_description/meshes/version3/STL/shoulder.stl" />
             </geometry>
         </visual>
@@ -53,5 +53,5 @@
             <origin xyz="0 0 0" rpy="0 ${PI/2} 0"/>
             <geometry>
-                <mesh filename="package://opr_description/meshes/version3/DAE/arm.dae" />
+                <mesh filename="package://opr_description/meshes/version3/STL/arm.stl" />
             </geometry>
         </visual>
@@ -72,5 +72,5 @@
             <origin xyz="0 0 0" rpy="${PI} 0 ${PI/2}"/>
             <geometry>
-                <mesh filename="package://opr_description/meshes/version3/DAE/hand.dae" />
+                <mesh filename="package://opr_description/meshes/version3/STL/hand.stl" />
             </geometry>
         </visual>

File: opr_description/urdf/version3/body/body.urdf.xacro (robot description, xacro)
@@ -17,5 +17,5 @@
             <origin xyz="0 0 0" rpy="${-PI/2} 0 ${PI/2}"/>
             <geometry>
-                <mesh filename="package://opr_description/meshes/version3/DAE/body.dae" />
+                <mesh filename="package://opr_description/meshes/version3/STL/body.stl" />
             </geometry>
         </visual>

File: opr_description/urdf/version3/head/head.urdf.xacro (robot description, xacro)
@@ -19,5 +19,5 @@
             <origin xyz="0 0 0" rpy="${-PI/2} ${PI/2} 0"/>
             <geometry>
-                <mesh filename="package://opr_description/meshes/version3/DAE/head.dae" />
+                <mesh filename="package://opr_description/meshes/version3/STL/head.stl" />
             </geometry>
         </visual>

File: opr_description/urdf/version3/legs/left_leg.urdf.xacro (robot description, xacro)
@@ -99,5 +99,5 @@
             <origin xyz="0 0 0" rpy="${-PI/2} 0 ${PI/2}"/>
             <geometry>
-                <mesh filename="package://opr_description/meshes/version3/DAE/waist_yaw.dae" />
+                <mesh filename="package://opr_description/meshes/version3/STL/waist_yaw.stl" />
             </geometry>
         </visual>
@@ -118,5 +118,5 @@
             <origin xyz="0 0 0" rpy="${-PI/2} ${-PI/2} 0"/>
             <geometry>
-                <mesh filename="package://opr_description/meshes/version3/DAE/waist_roll_left.dae" />
+                <mesh filename="package://opr_description/meshes/version3/STL/waist_roll_left.stl" />
             </geometry>
         </visual>
@@ -137,5 +137,5 @@
             <origin xyz="0 0 0" rpy="${PI/2} 0 ${-PI/2}"/>
             <geometry>
-                <mesh filename="package://opr_description/meshes/version3/DAE/slider_crank.dae" />
+                <mesh filename="package://opr_description/meshes/version3/STL/slider_crank.stl" />
             </geometry>
         </visual>
@@ -156,5 +156,5 @@
             <origin xyz="0 0 0" rpy="0 0 ${-PI/2}"/>
             <geometry>
-                <mesh filename="package://opr_description/meshes/version3/DAE/waist_pitch.dae" />
+                <mesh filename="package://opr_description/meshes/version3/STL/waist_pitch.stl" />
             </geometry>
         </visual>
@@ -175,5 +175,5 @@
             <origin xyz="0 0 0" rpy="0 0 ${PI/2}"/>
             <geometry>
-                <mesh filename="package://opr_description/meshes/version3/DAE/waist_pitch_mimic.dae" />
+                <mesh filename="package://opr_description/meshes/version3/STL/waist_pitch_mimic.stl" />
             </geometry>
         </visual>
@@ -194,5 +194,5 @@
             <origin xyz="0 0 0" rpy="0 ${PI} 0"/>
             <geometry>
-                <mesh filename="package://opr_description/meshes/version3/DAE/knee_pitch_left.dae" />
+                <mesh filename="package://opr_description/meshes/version3/STL/knee_pitch_left.stl" />
             </geometry>
         </visual>
@@ -213,5 +213,5 @@
             <origin xyz="0 0 0" rpy="0 0 ${-PI/2}"/>
             <geometry>
-                <mesh filename="package://opr_description/meshes/version3/DAE/shin_pitch.dae" />
+                <mesh filename="package://opr_description/meshes/version3/STL/shin_pitch.stl" />
             </geometry>
         </visual>
@@ -232,5 +232,5 @@
             <origin xyz="0 0 0" rpy="${PI} 0 ${PI/2}"/>
             <geometry>
-                <mesh filename="package://opr_description/meshes/version3/DAE/shin_pitch_mimic.dae" />
+                <mesh filename="package://opr_description/meshes/version3/STL/shin_pitch_mimic.stl" />
             </geometry>
         </visual>
@@ -251,5 +251,5 @@
             <origin xyz="0 0 0" rpy="${PI/2} 0 ${PI}"/>
             <geometry>
-                <mesh filename="package://opr_description/meshes/version3/DAE/independent_pitch.dae" />
+                <mesh filename="package://opr_description/meshes/version3/STL/independent_pitch.stl" />
             </geometry>
         </visual>
@@ -270,5 +270,5 @@
             <origin xyz="0 0 0" rpy="0 0 ${-PI/2}"/>
             <geometry>
-                <mesh filename="package://opr_description/meshes/version3/DAE/ankle_pitch_left.dae" />
+                <mesh filename="package://opr_description/meshes/version3/STL/ankle_pitch_left.stl" />
             </geometry>
         </visual>
@@ -289,5 +289,5 @@
             <origin xyz="0 0 0" rpy="${-PI/2} ${-PI/2} 0"/>
             <geometry>
-                <mesh filename="package://opr_description/meshes/version3/DAE/ankle_roll_left.dae" />
+                <mesh filename="package://opr_description/meshes/version3/STL/ankle_roll_left.stl" />
             </geometry>
         </visual>

File: opr_description/urdf/version3/legs/right_leg.urdf.xacro (robot description, xacro)
@@ -99,5 +99,5 @@
             <origin xyz="0 0 0" rpy="${-PI/2} 0 ${PI/2}"/>
             <geometry>
-                <mesh filename="package://opr_description/meshes/version3/DAE/waist_yaw.dae" />
+                <mesh filename="package://opr_description/meshes/version3/STL/waist_yaw.stl" />
             </geometry>
         </visual>
@@ -118,5 +118,5 @@
             <origin xyz="0 0 0" rpy="${-PI/2} ${-PI/2} 0"/>
             <geometry>
-                <mesh filename="package://opr_description/meshes/version3/DAE/waist_roll_right.dae" />
+                <mesh filename="package://opr_description/meshes/version3/STL/waist_roll_right.stl" />
             </geometry>
         </visual>
@@ -137,5 +137,5 @@
             <origin xyz="0 0 0" rpy="${PI/2} 0 ${-PI/2}"/>
             <geometry>
-                <mesh filename="package://opr_description/meshes/version3/DAE/slider_crank.dae" />
+                <mesh filename="package://opr_description/meshes/version3/STL/slider_crank.stl" />
             </geometry>
         </visual>
@@ -156,5 +156,5 @@
             <origin xyz="0 0 0" rpy="0 0 ${-PI/2}"/>
             <geometry>
-                <mesh filename="package://opr_description/meshes/version3/DAE/waist_pitch.dae" />
+                <mesh filename="package://opr_description/meshes/version3/STL/waist_pitch.stl" />
             </geometry>
         </visual>
@@ -175,5 +175,5 @@
             <origin xyz="0 0 0" rpy="0 0 ${PI/2}"/>
             <geometry>
-                <mesh filename="package://opr_description/meshes/version3/DAE/waist_pitch_mimic.dae" />
+                <mesh filename="package://opr_description/meshes/version3/STL/waist_pitch_mimic.stl" />
             </geometry>
         </visual>
@@ -194,5 +194,5 @@
             <origin xyz="0 0 0" rpy="${PI} ${PI} 0"/>
             <geometry>
-                <mesh filename="package://opr_description/meshes/version3/DAE/knee_pitch_right.dae" />
+                <mesh filename="package://opr_description/meshes/version3/STL/knee_pitch_right.stl" />
             </geometry>
         </visual>
@@ -213,5 +213,5 @@
             <origin xyz="0 0 0" rpy="0 0 ${-PI/2}"/>
             <geometry>
-                <mesh filename="package://opr_description/meshes/version3/DAE/shin_pitch.dae" />
+                <mesh filename="package://opr_description/meshes/version3/STL/shin_pitch.stl" />
             </geometry>
         </visual>
@@ -232,5 +232,5 @@
             <origin xyz="0 0 0" rpy="${PI} 0 ${PI/2}"/>
             <geometry>
-                <mesh filename="package://opr_description/meshes/version3/DAE/shin_pitch_mimic.dae" />
+                <mesh filename="package://opr_description/meshes/version3/STL/shin_pitch_mimic.stl" />
             </geometry>
         </visual>
@@ -251,5 +251,5 @@
             <origin xyz="0 0 0" rpy="${PI/2} 0 ${PI}"/>
             <geometry>
-                <mesh filename="package://opr_description/meshes/version3/DAE/independent_pitch.dae" />
+                <mesh filename="package://opr_description/meshes/version3/STL/independent_pitch.stl" />
             </geometry>
         </visual>
@@ -270,5 +270,5 @@
             <origin xyz="0 0 0" rpy="0 0 ${-PI/2}"/>
             <geometry>
-                <mesh filename="package://opr_description/meshes/version3/DAE/ankle_pitch_right.dae" />
+                <mesh filename="package://opr_description/meshes/version3/STL/ankle_pitch_right.stl" />
             </geometry>
         </visual>
@@ -289,5 +289,5 @@
             <origin xyz="0 0 0" rpy="${-PI/2} ${-PI/2} 0"/>
             <geometry>
-                <mesh filename="package://opr_description/meshes/version3/DAE/ankle_roll_right.dae" />
+                <mesh filename="package://opr_description/meshes/version3/STL/ankle_roll_right.stl" />
             </geometry>
         </visual>

Commit message: modify velocity

File: opr_description/urdf/version3/arms/left_arm.urdf.xacro (robot description, xacro)
@@ -6,5 +6,5 @@
         <child link="left_shoulder_link" />
         <origin xyz="0.0 0.06 0.072" rpy="${-PI/2} 0 0" />
-        <limit effort="1000" lower="${-3*PI/4}" upper="${3*PI/4}" velocity="1.0" />
+        <limit effort="1000" lower="${-3*PI/4}" upper="${3*PI/4}" velocity="4.8" />
         <axis xyz="0 0 1" />
     </joint>
@@ -13,5 +13,5 @@
         <child link="left_upper_arm_link" />
         <origin xyz="0 0 0.0315" rpy="0 ${PI/2} 0" />
-        <limit effort="1000" lower="0" upper="${PI}" velocity="1.0" />
+        <limit effort="1000" lower="0" upper="${PI}" velocity="4.8" />
         <axis xyz="0 0 1" />
     </joint>
@@ -20,5 +20,5 @@
         <child link="left_lower_arm_link" />
         <origin xyz="0 0.109 0" rpy="0 ${-PI/2} 0" />
-        <limit effort="1000" lower="${-3*PI/4}" upper="${3*PI/4}" velocity="1.0" />
+        <limit effort="1000" lower="${-3*PI/4}" upper="${3*PI/4}" velocity="4.8" />
         <axis xyz="0 0 1" />
     </joint>

File: opr_description/urdf/version3/arms/right_arm.urdf.xacro (robot description, xacro)
@@ -6,5 +6,5 @@
         <child link="right_shoulder_link" />
         <origin xyz="0.0 -0.06 0.072" rpy="${-PI/2} 0 0" />
-        <limit effort="1000" lower="${-3*PI/4}" upper="${3*PI/4}" velocity="1.0" />
+        <limit effort="1000" lower="${-3*PI/4}" upper="${3*PI/4}" velocity="4.8" />
         <axis xyz="0 0 1" />
     </joint>
@@ -13,5 +13,5 @@
         <child link="right_upper_arm_link" />
         <origin xyz="0 0 -0.0315" rpy="0 ${PI/2} 0" />
-        <limit effort="1000" lower="${-PI}" upper="0" velocity="1.0" />
+        <limit effort="1000" lower="${-PI}" upper="0" velocity="4.8" />
         <axis xyz="0 0 1" />
     </joint>
@@ -20,5 +20,5 @@
         <child link="right_lower_arm_link" />
         <origin xyz="0 0.109 0" rpy="0 ${-PI/2} 0" />
-        <limit effort="1000" lower="${-3*PI/4}" upper="${3*PI/4}" velocity="1.0" />
+        <limit effort="1000" lower="${-3*PI/4}" upper="${3*PI/4}" velocity="4.8" />
         <axis xyz="0 0 1" />
     </joint>

File: opr_description/urdf/version3/head/head.urdf.xacro (robot description, xacro)
@@ -6,5 +6,5 @@
         <child link="head_yaw_link" />
         <origin xyz="0 0 0.09475" rpy="0 0 0" />
-        <limit effort="1000" lower="${-3*PI/4}" upper="${3*PI/4}" velocity="1.0" />
+        <limit effort="1000" lower="${-3*PI/4}" upper="${3*PI/4}" velocity="4.8" />
         <axis xyz="0 0 1" />
     </joint>

File: opr_description/urdf/version3/legs/left_leg.urdf.xacro (robot description, xacro)
@@ -6,5 +6,5 @@
         <child link="left_waist_yaw_link" />
         <origin xyz="0.005 0.044 -0.0725" rpy="0 0 0" />
-        <limit effort="1000" lower="${-3*PI/4}" upper="${3*PI/4}" velocity="1.0" />
+        <limit effort="1000" lower="${-3*PI/4}" upper="${3*PI/4}" velocity="4.8" />
         <axis xyz="0 0 1" />
     </joint>
@@ -13,5 +13,5 @@
         <child link="left_waist_roll_link" />
         <origin xyz="0.024975 0 -0.055" rpy="0 ${PI/2} 0" />
-        <limit effort="1000" lower="${-PI/4}" upper="${PI/4}" velocity="1.0" />
+        <limit effort="1000" lower="${-PI/4}" upper="${PI/4}" velocity="4.8" />
         <axis xyz="0 0 1" />
     </joint>
@@ -21,5 +21,5 @@
         <origin xyz="-0.018 0 -0.091475" rpy="0 0 0" />
         <mimic joint="left_waist_roll_joint" multiplier="-2" offset="0" />
-        <limit effort="1000" lower="${-PI/2}" upper="${PI/2}" velocity="2.0" />
+        <limit effort="1000" lower="${-PI/2}" upper="${PI/2}" velocity="4.8" />
         <axis xyz="0 0 1" />
     </joint>
@@ -28,5 +28,5 @@
         <child link="left_waist_pitch_link" />
         <origin xyz="0 0 -0.025" rpy="${-PI/2} 0 0" />
-        <limit effort="1000" lower="${-PI/2}" upper="${PI/6}" velocity="1.0" />
+        <limit effort="1000" lower="${-PI/2}" upper="${PI/6}" velocity="4.8" />
         <axis xyz="0 0 1" />
     </joint>
@@ -36,5 +36,5 @@
         <origin xyz="0.02 0 -0.057" rpy="${-PI/2} 0 0" />
         <mimic joint="left_waist_pitch_joint" multiplier="1" offset="0" />
-        <limit effort="1000" lower="${-PI/2}" upper="${PI/6}" velocity="1.0" />
+        <limit effort="1000" lower="${-PI/2}" upper="${PI/6}" velocity="4.8" />
         <axis xyz="0 0 1" />
     </joint>
@@ -44,5 +44,5 @@
         <origin xyz="0.1 0 0" rpy="0 0 0" />
         <mimic joint="left_waist_pitch_joint" multiplier="-1" offset="0" />
-        <limit effort="1000" lower="${-PI/6}" upper="${PI/2}" velocity="1.0" />
+        <limit effort="1000" lower="${-PI/6}" upper="${PI/2}" velocity="4.8" />
         <axis xyz="0 0 1" />
     </joint>
@@ -51,5 +51,5 @@
         <child link="left_shin_pitch_link" />
         <origin xyz="0.057 0 0" rpy="0 0 0" />
-        <limit effort="1000" lower="${-PI/6}" upper="${PI/2}" velocity="1.0" />
+        <limit effort="1000" lower="${-PI/6}" upper="${PI/2}" velocity="4.8" />
         <axis xyz="0 0 1" />
     </joint>
@@ -59,5 +59,5 @@
         <origin xyz="0.037 0.032 0" rpy="0 0 0" />
         <mimic joint="left_knee_pitch_joint" multiplier="1" offset="0" />
-        <limit effort="1000" lower="${-PI/6}" upper="${PI/2}" velocity="1.0" />
+        <limit effort="1000" lower="${-PI/6}" upper="${PI/2}" velocity="4.8" />
         <axis xyz="0 0 1" />
     </joint>
@@ -67,5 +67,5 @@
         <origin xyz="0.1 0 0" rpy="0 0 0" />
         <mimic joint="left_knee_pitch_joint" multiplier="-1" offset="0" />
-        <limit effort="1000" lower="${-PI/2}" upper="${PI/2}" velocity="1.0" />
+        <limit effort="1000" lower="${-PI/2}" upper="${PI/2}" velocity="4.8" />
         <axis xyz="0 0 1" />
     </joint>
@@ -74,5 +74,5 @@
         <child link="left_ankle_pitch_link" />
         <origin xyz="0.0001 0 0" rpy="0 0 0" />
-        <limit effort="1000" lower="${-3*PI/4}" upper="${3*PI/4}" velocity="1.0" />
+        <limit effort="1000" lower="${-3*PI/4}" upper="${3*PI/4}" velocity="4.8" />
         <axis xyz="0 0 1" />
     </joint>
@@ -81,5 +81,5 @@
         <child link="left_ankle_roll_link" />
         <origin xyz="0 0.0325 0" rpy="${PI/2} 0 0"/>
-        <limit effort="1000" lower="${-PI/2}" upper="${PI/2}" velocity="1.0" />
+        <limit effort="1000" lower="${-PI/2}" upper="${PI/2}" velocity="4.8" />
         <axis xyz="0 0 1" />
     </joint>

File: opr_description/urdf/version3/legs/leg.gazebo.xacro (robot description, xacro)
@@ -18,5 +18,5 @@
             <mu1>1.0</mu1>
             <mu2>1.0</mu2>
-            <kp>1000000.0</kp>
+            <kp>10000.0</kp>
             <kd>100.0</kd>
             <gravity>false</gravity>

File: opr_description/urdf/version3/legs/right_leg.urdf.xacro (robot description, xacro)
@@ -6,5 +6,5 @@
         <child link="right_waist_yaw_link" />
         <origin xyz="0.005 -0.044 -0.0725" rpy="0 0 0" />
-        <limit effort="1000" lower="${-3*PI/4}" upper="${3*PI/4}" velocity="1.0" />
+        <limit effort="1000" lower="${-3*PI/4}" upper="${3*PI/4}" velocity="4.8" />
         <axis xyz="0 0 1" />
     </joint>
@@ -13,5 +13,5 @@
         <child link="right_waist_roll_link" />
         <origin xyz="0.024975 0 -0.055" rpy="0 ${PI/2} 0" />
-        <limit effort="1000" lower="${-PI/4}" upper="${PI/4}" velocity="1.0" />
+        <limit effort="1000" lower="${-PI/4}" upper="${PI/4}" velocity="4.8" />
         <axis xyz="0 0 1" />
     </joint>
@@ -21,5 +21,5 @@
         <origin xyz="-0.018 0 -0.091475" rpy="0 0 0" />
         <mimic joint="right_waist_roll_joint" multiplier="-2" offset="0" />
-        <limit effort="1000" lower="${-PI/2}" upper="${PI/2}" velocity="2.0" />
+        <limit effort="1000" lower="${-PI/2}" upper="${PI/2}" velocity="4.8" />
         <axis xyz="0 0 1" />
     </joint>
@@ -28,5 +28,5 @@
         <child link="right_waist_pitch_link" />
         <origin xyz="0 0 -0.025" rpy="${-PI/2} 0 0" />
-        <limit effort="1000" lower="${-PI/2}" upper="${PI/6}" velocity="1.0" />
+        <limit effort="1000" lower="${-PI/2}" upper="${PI/6}" velocity="4.8" />
         <axis xyz="0 0 1" />
     </joint>
@@ -36,5 +36,5 @@
         <origin xyz="0.02 0 -0.057" rpy="${-PI/2} 0 0" />
         <mimic joint="right_waist_pitch_joint" multiplier="1" offset="0" />
-        <limit effort="1000" lower="${-PI/2}" upper="${PI/6}" velocity="1.0" />
+        <limit effort="1000" lower="${-PI/2}" upper="${PI/6}" velocity="4.8" />
         <axis xyz="0 0 1" />
     </joint>
@@ -44,5 +44,5 @@
         <origin xyz="0.1 0 0" rpy="0 0 0" />
         <mimic joint="right_waist_pitch_joint" multiplier="-1" offset="0" />
-        <limit effort="1000" lower="${-PI/6}" upper="${PI/2}" velocity="1.0" />
+        <limit effort="1000" lower="${-PI/6}" upper="${PI/2}" velocity="4.8" />
         <axis xyz="0 0 1" />
     </joint>
@@ -51,5 +51,5 @@
         <child link="right_shin_pitch_link" />
         <origin xyz="0.057 0 0" rpy="0 0 0" />
-        <limit effort="1000" lower="${-PI/6}" upper="${PI/2}" velocity="1.0" />
+        <limit effort="1000" lower="${-PI/6}" upper="${PI/2}" velocity="4.8" />
         <axis xyz="0 0 1" />
     </joint>
@@ -59,5 +59,5 @@
         <origin xyz="0.037 0.032 0" rpy="0 0 0" />
         <mimic joint="right_knee_pitch_joint" multiplier="1" offset="0" />
-        <limit effort="1000" lower="${-PI/6}" upper="${PI/2}" velocity="1.0" />
+        <limit effort="1000" lower="${-PI/6}" upper="${PI/2}" velocity="4.8" />
         <axis xyz="0 0 1" />
     </joint>
@@ -67,5 +67,5 @@
         <origin xyz="0.1 0 0" rpy="0 0 0" />
         <mimic joint="right_knee_pitch_joint" multiplier="-1" offset="0" />
-        <limit effort="1000" lower="${-PI/2}" upper="${PI/2}" velocity="1.0" />
+        <limit effort="1000" lower="${-PI/2}" upper="${PI/2}" velocity="4.8" />
         <axis xyz="0 0 1" />
     </joint>
@@ -74,5 +74,5 @@
         <child link="right_ankle_pitch_link" />
         <origin xyz="0.0001 0 0" rpy="0 0 0" />
-        <limit effort="1000" lower="${-3*PI/4}" upper="${3*PI/4}" velocity="1.0" />
+        <limit effort="1000" lower="${-3*PI/4}" upper="${3*PI/4}" velocity="4.8" />
         <axis xyz="0 0 1" />
     </joint>
@@ -81,5 +81,5 @@
         <child link="right_ankle_roll_link" />
         <origin xyz="0 0.0325 0" rpy="${PI/2} 0 0"/>
-        <limit effort="1000" lower="${-PI/2}" upper="${PI/2}" velocity="1.0" />
+        <limit effort="1000" lower="${-PI/2}" upper="${PI/2}" velocity="4.8" />
         <axis xyz="0 0 1" />
     </joint>
